File: Hardware/SongBeam 3.1_kicad/SongBeam4.0/SongBeam4.0.kicad_pcb (KiCad board)
At the start: 0 parts

Commit message: pcb sketch v1
Parts:
- added BAT1: 3034, 79523211:79523211, F.Cu at (276.3, 105.6)
- added C1: 100nF, Capacitor_SMD:C_0805_2012Metric, F.Cu at (15.2, 20.0)
- added C10: 47pF, Capacitor_SMD:C_0805_2012Metric, F.Cu at (20.0, 47.9)
- added C11: 100nF, Capacitor_SMD:C_0805_2012Metric, F.Cu at (62.4, 42.5)
- added C12: 47pF, Capacitor_SMD:C_0805_2012Metric, F.Cu at (67.2, 48.0)
- added C13: 100nF, Capacitor_SMD:C_0805_2012Metric, F.Cu at (15.2, 55.6)
- added C14: 47pF, Capacitor_SMD:C_0805_2012Metric, F.Cu at (20.0, 60.9)
- added C15: 100nF, Capacitor_SMD:C_0805_2012Metric, F.Cu at (62.4, 55.5)
- added C16: 47pF, Capacitor_SMD:C_0805_2012Metric, F.Cu at (67.1, 60.9)
- added C17: 1uF, Capacitor_SMD:C_0805_2012Metric, F.Cu at (137.7, 162.4)
- added C18: 100nF, Capacitor_SMD:C_0805_2012Metric, F.Cu at (137.7, 165.4)
- added C19: 1uF, Capacitor_SMD:C_0805_2012Metric, F.Cu at (137.7, 168.5)
- added C2: 47pF, Capacitor_SMD:C_0805_2012Metric, F.Cu at (20.0, 25.4)
- added C20: 1uF, Capacitor_SMD:C_0805_2012Metric, F.Cu at (137.7, 171.5)
- added C21: 100nF, Capacitor_SMD:C_0805_2012Metric, F.Cu at (137.7, 174.5)
- added C22: 10uF, Capacitor_SMD:C_0805_2012Metric, F.Cu at (137.7, 177.5)
- added C23: 10uF, Capacitor_SMD:C_0805_2012Metric, F.Cu at (137.7, 180.5)
- added C24: 100nF, Capacitor_SMD:C_0805_2012Metric, F.Cu at (137.7, 183.5)
- added C25: 100nF, Capacitor_SMD:C_0805_2012Metric, F.Cu at (154.5, 177.8)
- added C26: 10uF, Capacitor_SMD:C_0805_2012Metric, F.Cu at (154.5, 180.8)
- added C27: 22uF, Capacitor_SMD:C_0805_2012Metric, F.Cu at (28.4, 103.1)
- added C28: 22uF, Capacitor_SMD:C_0805_2012Metric, F.Cu at (59.1, 112.5)
- added C29: 1uF, Capacitor_SMD:C_0805_2012Metric, F.Cu at (59.1, 115.5)
- added C3: 100nF, Capacitor_SMD:C_0805_2012Metric, F.Cu at (62.3, 20.0)
- added C32: 100nF, Capacitor_SMD:C_0805_2012Metric, F.Cu at (59.1, 118.5)
- added C33: 1000nF, Capacitor_SMD:C_0201_0603Metric, F.Cu at (63.4, 126.9)
- added C34: 0.1uF, Capacitor_SMD:C_0805_2012Metric, F.Cu at (201.2, 160.5)
- added C35: 0.1uF, Capacitor_SMD:C_0805_2012Metric, F.Cu at (201.2, 163.5)
- added C38: 22uF, Capacitor_SMD:C_0805_2012Metric, F.Cu at (24.4, 94.6)
- added C39: 56pF, Capacitor_SMD:C_0201_0603Metric, F.Cu at (214.3, 138.0)
- added C4: 47pF, Capacitor_SMD:C_0805_2012Metric, F.Cu at (67.1, 25.4)
- added C40: 10µF, Capacitor_SMD:C_0805_2012Metric, F.Cu at (63.6, 106.4)
- added C41: 4.7µF, Capacitor_SMD:C_0805_2012Metric, F.Cu at (63.6, 109.4)
- added C43: 1µF, Capacitor_SMD:C_0805_2012Metric, F.Cu at (102.2, 143.0)
- added C44: 1µF, Capacitor_SMD:C_0805_2012Metric, F.Cu at (102.2, 146.0)
- added C5: 100nF, Capacitor_SMD:C_0805_2012Metric, F.Cu at (15.2, 30.6)
- added C6: 47pF, Capacitor_SMD:C_0805_2012Metric, F.Cu at (19.9, 35.9)
- added C7: 100nF, Capacitor_SMD:C_0805_2012Metric, F.Cu at (62.4, 30.6)
- added C8: 47pF, Capacitor_SMD:C_0805_2012Metric, F.Cu at (67.1, 35.9)
- added C9: 100nF, Capacitor_SMD:C_0805_2012Metric, F.Cu at (15.2, 42.5)
- added CHG1: ORANGE, LED_SMD:LED_0201_0603Metric, F.Cu at (35.6, 108.1)
- added D1: APHF1608LSEEQBDZGKC, LED_SMD:LED-APA102-2020, F.Cu at (239.3, 104.2)
- added D2: BAT54AW, Package_TO_SOT_SMD:SOT-323_SC-70, F.Cu at (249.3, 132.9)
- added D4: MBRX120, MBRX120LF:SOD3716X135N, F.Cu at (45.2, 111.2)
- added D5: MBRX120, MBRX120LF:SOD3716X135N, F.Cu at (46.2, 116.1)
- added D6: MBRX120, MBRX120LF:SOD3716X135N, F.Cu at (24.7, 89.8)
- added D7: BZV55B5V1, Diode_SMD:D_MiniMELF, F.Cu at (28.0, 89.8)
- added F3: Polyfuse, MINISMDC050F-2:MINISMDC050F2, F.Cu at (98.0, 132.0)
- added FAULT1: RED, LED_SMD:LED_0201_0603Metric, F.Cu at (32.8, 112.4)
- added J1: Conn_01x02, Connector_PinHeader_1.00mm:PinHeader_1x02_P1.00mm_Horizontal, F.Cu at (140.1, 15.6)
- added J10: 732511150, DFE201612E:1286ASH1R0MP2, F.Cu at (91.8, 91.5)
- added J11: USB_B_Micro, 10118192:101181920002LF, F.Cu at (19.0, 92.0)
- added J12: Conn_01x02, Connector_PinHeader_1.00mm:PinHeader_1x02_P1.00mm_Horizontal, F.Cu at (21.5, 84.8)
- added J13: Conn_01x02, Connector_PinHeader_1.00mm:PinHeader_1x02_P1.00mm_Horizontal, F.Cu at (25.0, 99.1)
- added J2: RJ45, RJHSE-3380:CONN_RJHSE-3380_AMP, F.Cu at (301.1, 96.7)
- added J3: RJ45, RJHSE-3380:CONN_RJHSE-3380_AMP, F.Cu at (301.1, 77.2)
- added J4: Conn_01x07, Connector_PinHeader_1.00mm:PinHeader_1x07_P1.00mm_Horizontal, F.Cu at (148.1, -4.33)
- added J5: Conn_01x04, Connector_PinHeader_1.00mm:PinHeader_1x04_P1.00mm_Horizontal, F.Cu at (83.4, 30.1)
- added J6: Conn_01x07, Connector_PinHeader_1.00mm:PinHeader_1x07_P1.00mm_Horizontal, F.Cu at (135.4, -0.28)
- added J7: Conn_01x09, Connector_PinHeader_1.00mm:PinHeader_1x09_P1.00mm_Horizontal, F.Cu at (140.1, 27.7)
- added J8: Conn_01x04, Connector_PinHeader_1.00mm:PinHeader_1x04_P1.00mm_Horizontal, F.Cu at (130.2, 14.4)
- added J9: Conn_01x08, Connector_PinHeader_1.00mm:PinHeader_1x08_P1.00mm_Horizontal, F.Cu at (227.4, 139.9)
- added JP1: SolderJumper_2_Bridged, Jumper:SolderJumper-2_P1.3mm_Bridged_RoundedPad1.0x1.5mm, F.Cu at (107.2, 123.9)
- added L1: DFE201612E-2R2M=P2, DFE201612E:1286ASH1R0MP2, F.Cu at (91.8, 94.8)
- added L2: 27nH, LQM2HPZ2R2MG0L:LQM2HPN1R0MG0L, F.Cu at (219.6, 138.5)
- added R1: 100R, Resistor_SMD:R_0805_2012Metric, F.Cu at (16.1, 23.1)
- added R10: 100K, Resistor_SMD:R_0805_2012Metric, F.Cu at (20.0, 45.6)
- added R11: 100R, Resistor_SMD:R_0805_2012Metric, F.Cu at (63.4, 45.7)
- added R12: 100K, Resistor_SMD:R_0805_2012Metric, F.Cu at (67.2, 45.7)
- added R13: 100R, Resistor_SMD:R_0805_2012Metric, F.Cu at (16.3, 58.7)
- added R14: 100K, Resistor_SMD:R_0805_2012Metric, F.Cu at (20.0, 58.7)
- added R15: 100R, Resistor_SMD:R_0805_2012Metric, F.Cu at (63.3, 58.6)
- added R16: 100K, Resistor_SMD:R_0805_2012Metric, F.Cu at (67.1, 58.6)
- added R17: 100R, Resistor_SMD:R_0805_2012Metric, F.Cu at (165.5, 174.0)
- added R18: 330R, Resistor_SMD:R_0805_2012Metric, F.Cu at (254.1, 98.8)
- added R19: 330R, Resistor_SMD:R_0805_2012Metric, F.Cu at (254.1, 101.7)
- added R2: 100R, Resistor_SMD:R_0805_2012Metric, F.Cu at (20.0, 23.1)
- added R20: 750R, Resistor_SMD:R_0805_2012Metric, F.Cu at (254.1, 104.7)
- added R21: 1K, Resistor_SMD:R_0805_2012Metric, F.Cu at (27.7, 100.1)
- added R22: 10K, Resistor_SMD:R_0805_2012Metric, F.Cu at (30.0, 100.1)
- added R23: 1K, Resistor_SMD:R_0805_2012Metric, F.Cu at (35.0, 100.7)
- added R24: 300, Resistor_SMD:R_0805_2012Metric, F.Cu at (28.2, 115.6)
- added R25: 6.8K, Resistor_SMD:R_0805_2012Metric, F.Cu at (26.1, 77.7)
- added R26: 5.1K, Resistor_SMD:R_0805_2012Metric, F.Cu at (35.3, 77.8)
- added R27: 10K, Resistor_SMD:R_0805_2012Metric, F.Cu at (80.9, 118.8)
- added R28: 100K, Resistor_SMD:R_0805_2012Metric, F.Cu at (80.9, 121.8)
- added R29: 100K, Resistor_SMD:R_0805_2012Metric, F.Cu at (80.9, 124.8)
- added R3: 100R, Resistor_SMD:R_0805_2012Metric, F.Cu at (63.3, 23.1)
- added R30: 1M, Resistor_SMD:R_0805_2012Metric, F.Cu at (80.9, 127.7)
- added R31: 105K, Resistor_SMD:R_0805_2012Metric, F.Cu at (80.9, 130.7)
- added R33: 100K, Resistor_SMD:R_0805_2012Metric, F.Cu at (80.9, 133.6)
- added R34: 1k, Resistor_SMD:R_0805_2012Metric, F.Cu at (86.4, 112.6)
- added R35: 100k, Resistor_SMD:R_0805_2012Metric, F.Cu at (86.4, 115.5)
- added R36: NC, Resistor_SMD:R_0805_2012Metric, F.Cu at (85.3, 118.8)
- added R37: 1M, Resistor_SMD:R_0805_2012Metric, F.Cu at (85.3, 121.8)
- added R38: 10K, Resistor_SMD:R_0805_2012Metric, F.Cu at (196.1, 156.8)
- added R39: 100k, Resistor_SMD:R_0805_2012Metric, F.Cu at (217.6, 129.7)
- added R4: 100K, Resistor_SMD:R_0805_2012Metric, F.Cu at (67.1, 23.1)
- added R40: 267K, Resistor_SMD:R_0805_2012Metric, F.Cu at (85.3, 130.7)
- added R5: 100R, Resistor_SMD:R_0805_2012Metric, F.Cu at (16.2, 33.7)
- added R6: 100K, Resistor_SMD:R_0805_2012Metric, F.Cu at (19.9, 33.7)
- added R7: 100R, Resistor_SMD:R_0805_2012Metric, F.Cu at (63.3, 33.6)
- added R8: 100K, Resistor_SMD:R_0805_2012Metric, F.Cu at (67.1, 33.6)
- added R9: 100R, Resistor_SMD:R_0805_2012Metric, F.Cu at (16.3, 45.6)
- added S2: SLW-12689-4A-N-D, SLW12689:SLW126894AND, F.Cu at (27.9, 82.9)
- added SW2: PTS815 SJM 250 SMTR LFS, PTS815:SW4_PTS815 SJM 250 SMTR LFS_CNK, F.Cu at (125.1, 105.4)
- added SW3: PTS815 SJM 250 SMTR LFS, PTS815:SW4_PTS815 SJM 250 SMTR LFS_CNK, F.Cu at (283.9, 65.2)
- added TP1: TestPoint, TestPoint:TestPoint_Pad_D1.0mm, F.Cu at (50.8, 111.0)
- added TP2: TestPoint, TestPoint:TestPoint_Pad_D1.0mm, F.Cu at (55.0, 115.3)
- added TP7: TestPoint, TestPoint:TestPoint_Pad_D1.0mm, F.Cu at (98.3, 142.9)
- added TP8: TestPoint, TestPoint:TestPoint_Pad_D1.0mm, F.Cu at (98.3, 145.9)
- added U1: IM66D132H, mics:IFX-PG-TLGA-5N-9-V, F.Cu at (18.8, 19.6)
- added U10: Teensy4.1, Teensy:Teensy41, F.Cu at (249.5, 80.9)
- added U11: BQ25185, BQ25185DLHR:BQ25185DLHR, F.Cu at (27.5, 94.8)
- added U12: AO6604, AO6604:AO6604, F.Cu at (91.7, 82.1)
- added U13: TPS62842DGRR, TPS6284:TPS62842DGRR, F.Cu at (64.7, 92.5)
- added U14: TPL5111DDCR, TPL5111DDCR:TPL5111DDCR, F.Cu at (105.9, 113.3)
- added U15: AO6604, AO6604:AO6604, F.Cu at (98.8, 89.6)
- added U16: TXS0108EPW, Package_SO:TSSOP-20_4.4x6.5mm_P0.65mm, F.Cu at (189.5, 163.5)
- added U17: LP5907MFX-1.8/NOPB, ul_LP5907MFX-1-2-NOPB:DBV0005A_N, F.Cu at (88.2, 144.8)
- added U18: AO3407A, AO3407A:SOT-23-3L_AOS, F.Cu at (236.2, 130.2)
- added U19: MAX-M10M-00B, MAX-M10M:MAX-M10M-00B, F.Cu at (226.2, 126.7)
- added U2: IM66D132H, mics:IFX-PG-TLGA-5N-9-V, F.Cu at (66.0, 19.6)
- added U3: IM66D132H, mics:IFX-PG-TLGA-5N-9-V, F.Cu at (18.8, 30.2)
- added U4: IM66D132H, mics:IFX-PG-TLGA-5N-9-V, F.Cu at (65.9, 30.1)
- added U5: IM66D132H, mics:IFX-PG-TLGA-5N-9-V, F.Cu at (18.8, 42.1)
- added U6: IM66D132H, mics:IFX-PG-TLGA-5N-9-V, F.Cu at (66.0, 42.1)
- added U7: IM66D132H, mics:IFX-PG-TLGA-5N-9-V, F.Cu at (18.8, 55.1)
- added U8: IM66D132H, mics:IFX-PG-TLGA-5N-9-V, F.Cu at (66.0, 55.1)
- added U9: PCMD3180IRTWR, PCMD3180IRTWR:PCMD3180IRTWR, F.Cu at (153.1, 158.6)
Other:
- copper layers 0 -> 2
