File: Hardware/SongBeam 3.1_kicad/SongBeam4.0/SongBeam4.0.kicad_pcb (KiCad board)
At the start: 2 copper layers, 175.8 x 104.9 mm, 133 parts, among them J1 Conn_01x02, J10 732511150, J11 Conn_01x02, J12 Conn_01x02, J2 RJ45, J3 RJ45, J4 Conn_01x07, J5 Conn_01x04, J6 Conn_01x07, J7 Conn_01x04, J8 Conn_01x08, J9 USB_B_Micro, SW2 PTS815 SJM 250 SMTR LFS, SW3 PTS815 SJM 250 SMTR LFS, U1 IM66D132H, U10 Teensy4.1, U11 BQ25185DLHR, U12 AO6604, U13 TPS62842, U14 TPL5111DDCR, U15 AO6604, U16 TXS0108EPW, U17 LP5907MFX-1.8/NOPB, U18 AO3407A, U19 MAX-M10M-00B, U2 IM66D132H, U3 IM66D132H, U4 IM66D132H, U5 IM66D132H, U6 IM66D132H, U7 IM66D132H, U8 IM66D132H, U9 PCMD3180

Commit message: gerber
Parts:
- U11: value BQ25185DLHR -> WSON10_DLH_TEX
- U12, U15: value AO6604 -> TSOP6_AOS
- U19: value MAX-M10M-00B -> MOD18_MAX-M10M_UBL
- moved D1 2.19 mm to (125.5, 106.9)
- moved R18 2.19 mm to (130.3, 107.0)
- moved R19 2.19 mm to (133.4, 107.0)
- moved R20 2.19 mm to (136.6, 107.2)
- moved U10 1.94 mm to (134.9, 120.2)
- moved J10 1.73 mm to (73.5, 129.5)
- moved C10 1.47 mm to (56.6, 70.2)
- moved R10 1.47 mm to (56.6, 67.9)
- moved U5 1.47 mm to (55.5, 64.5)
- moved C9 1.47 mm to (51.9, 64.9)
- moved R9 1.47 mm to (52.9, 67.9)
- moved C8 0.67 mm to (166.7, 38.4)
- moved R8 0.67 mm to (166.7, 36.1)
- moved U4 0.67 mm to (165.6, 32.6)
- moved C7 0.67 mm to (162.0, 33.1)
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- renumbered REF** to REF1, REF** to REF2, REF** to REF3, REF** to REF4
Connections:
- U7 pad 2: +1V8 -> GND
Routing:
- net GND: track 1007.3 -> 1028.2 mm, vias 50 -> 54
- net +1V8: track 434.5 -> 420.7 mm, vias 19 -> 17
- net TXGPS: track 47.1 -> 39.3 mm
- net MCLK_TDM2_3.3V: track 99.1 -> 106.7 mm
- net +3.3V: track 162.9 -> 168.6 mm
- net Net-(D1-Pad1): track 55.5 -> 50.2 mm
- net RXGPS: track 41.4 -> 36.4 mm
- net GPS_PWR: track 75.1 -> 70.4 mm, vias 1 -> 2
- net Net-(U10-VBAT): track 54.6 -> 59.3 mm, vias 0 -> 2
- net micGRP_4out_1.8V: track 73.7 -> 78.3 mm, vias 2 -> 3
- net Net-(D1-Pad4): track 10.6 -> 6.41 mm, vias 2 -> 0
- net sensorSCL: track 55.7 -> 59.2 mm
- net OUTPUT_TDM1_3.3V: track 53.7 -> 51.0 mm, vias 2 -> 1
- net Net-(U10-16_A2_RX4_SCL1): track 28.4 -> 26.0 mm
- net PWR: track 123.2 -> 125.5 mm, vias 1 -> 0
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Other:
- board text added: "Myadestes melanops"
