File: Hardware/SongBeam 3.1_kicad/SongBeam4.0/SongBeam4.0.kicad_pcb (KiCad board)
At the start: 2 copper layers, 175.8 x 104.9 mm, 133 parts, among them J1 Conn_01x02, J10 732511150, J11 Conn_01x02, J12 Conn_01x02, J2 RJ45, J3 RJ45, J4 Conn_01x07, J5 Conn_01x04, J6 Conn_01x07, J7 Conn_01x04, J8 Conn_01x08, J9 USB_B_Micro, SW2 PTS815 SJM 250 SMTR LFS, SW3 PTS815 SJM 250 SMTR LFS, U1 IM66D132H, U10 Teensy4.1, U11 WSON10_DLH_TEX, U12 TSOP6_AOS, U13 TPS62842, U14 TPL5111DDCR, U15 TSOP6_AOS, U16 TXS0108EPW, U17 LP5907MFX-1.8/NOPB, U18 AO3407A, U19 MOD18_MAX-M10M_UBL, U2 IM66D132H, U3 IM66D132H, U4 IM66D132H, U5 IM66D132H, U6 IM66D132H, U7 IM66D132H, U8 IM66D132H, U9 PCMD3180

Commit message: Layout updates
Parts:
- removed REF1, REF2, REF3, REF4: MountingHole_3.2mm_M3, MountingHole:MountingHole_3.2mm_M3
- added C30: 10nF, Capacitor_SMD:C_0201_0603Metric, F.Cu at (90.6, 126.8)
- added D8: MBRX120LF-TP, MBRX120LF:SOD3716X135N, F.Cu at (28.1, 108.5)
- C29: value 1uF -> 22uF
- C33: value 1000nF -> 100muF
- C39: value 56pF -> 47pF
- L2: value 27nH -> GJM1555C1H470JB01D; footprint LQM2HPZ2R2MG0L:LQM2HPN1R0MG0L -> GPSINDUCTOR:CAPC1005X55N
- U11: value WSON10_DLH_TEX -> BQ25185DLHR
- U12, U15: value TSOP6_AOS -> AO6604
- U13: value TPS62842 -> TPS62842DGRR
- U19: value MOD18_MAX-M10M_UBL -> MAX-M10M-00B
- U9: value PCMD3180 -> PCMD3180IRTWR
- moved C33 96.5 mm to (167.5, 128.1), turned to -90 degrees
Connections:
- C33 pad 1: GND -> PWR
- C33 pad 2: Net-(U15-G1) -> GND
- J11 pad 1: VBUS -> Net-(D8-A)
- U10 pad 7: unconnected-(U10-5_IN2-Pad7) -> TMPPS
- U7 pad 2: GND -> +1V8
Routing:
- net TMPPS: track 8.82 -> 93.9 mm, vias 0 -> 3
- net GND: track 1028.2 -> 1075.1 mm, vias 54 -> 52
- net Net-(D8-A): track 0.00 -> 7.30 mm, vias 0 -> 1
- net PWR: track 125.5 -> 131.8 mm, vias 0 -> 1
- net +5V: track 35.7 -> 40.4 mm
- net GPS_ON: track 77.3 -> 72.8 mm
- net VBUS: track 35.3 -> 38.9 mm, vias 1 -> 2
- net OUTPUT_TDM1_3.3V: track 51.0 -> 48.4 mm
- net antenna: track 19.7 -> 21.8 mm
- net Net-(U19-VCC_RF): track 6.14 -> 8.21 mm
- net +1V8: track 420.7 -> 422.7 mm
- net Net-(U18-D): track 14.7 -> 16.2 mm
- net Net-(U15-G1): track 14.7 -> 13.6 mm
- net RXGPS: track 36.4 -> 37.0 mm
- net emrg_pwr_swch: track 92.4 -> 92.2 mm, vias 2 -> 3
