File: Hardware/SongBeam 3.1_kicad/SongBeam4.0/SongBeam4.0.kicad_sch (KiCad schematic)
At the start: 127 parts, among them IC3 TPS62842DGRR, J1 Conn_01x02, J10 RJ45, J11 Conn_01x04, J2 Conn_01x04, J3 JST2PH CONECTOR, J4 Conn_01x09, J6 USB_B_Micro, J7 Conn_01x07, J8 Conn_01x07, J9 RJ45, Q1 CPH6350-TL-W, Q2 AO6604, SW1 SW_SPDT, U1 PCMD3180IRTWR, U10 LP5907MFX-1.8_NOPB, U11 TPL5110, U12 TXS0108EPW, U13 Teensy4.1, U14 3034, U15 BQ25185DLHR, U2 IM66D132H, U3 IM66D132H, U4 IM66D132H, U5 IM66D132H, U6 IM66D132H, U7 IM66D132H, U8 IM66D132H, U9 IM66D132H

Commit message: V1 BRD_4.0
finish the schematics
Parts:
- removed C27, C28: 1µF, Capacitor_SMD:C_0805_2012Metric, symbol Device:C_Small
- removed C32: 4.7µF, Capacitor_SMD:C_0805_2012Metric, symbol Device:C_Small
- removed C33: 10µF, Capacitor_SMD:C_0805_2012Metric, symbol Device:C_Small
- removed F1: Polyfuse, LIB_MINISMDC110F-2:MINISMDC050F2, symbol Device:Polyfuse
- removed IC3: TPS62842DGRR, SOP65P490X110-9N, symbol SoundRecorder_2.0:TPS62842DGRR
- removed J3: JST2PH CONECTOR, symbol Connector:Conn_01x02_Socket
- removed Q2: AO6604, Package_SO:TSOP-6_1.65x3.05mm_P0.95mm, symbol SoundRecorder_2.0:AO6604
- removed R18, R38: 100K, Resistor_SMD:R_0805_2012Metric, symbol Device:R_Small
- removed R18: 1M, Resistor_SMD:R_0805_2012Metric, symbol Device:R_Small
- removed R20: 105K, Resistor_SMD:R_0805_2012Metric, symbol Device:R_Small
- removed R33: 267K, Resistor_SMD:R_0805_2012Metric, symbol Device:R_Small
- removed R42, R44, R47, R48, R49: 33R, Resistor_SMD:R_0805_2012Metric, symbol Device:R_Small
- removed R43, R46: 2.2K, Resistor_SMD:R_0805_2012Metric, symbol Device:R_Small
- removed R45: 10000K, Resistor_SMD:R_0805_2012Metric, symbol Device:R_Small
- removed S3: PTS815_SJM_250_SMTR_LFS, PTS815_SJM_250_SMTR_LFS:PTS815SJM250SMTRLFS, symbol SoundRecorder_2.0:PTS815_SJM_250_SMTR_LFS
- removed TP3, TP4: TestPoint, TestPoint:TestPoint_Pad_D1.0mm, symbol Connector:TestPoint
- removed U10: LP5907MFX-1.8_NOPB, ul_LP5907MFX-1-2-NOPB:LP5907MFX-1.2&slash_NOPB, symbol SoundRecorder_2.0:LP5907MFX-1.8_NOPB
- added C31, C32 (x2), C46: 100nF, Capacitor_SMD:C_0805_2012Metric, symbol Device:C_Small
- added C33 (x2), C47: 1000nF, symbol Device:C_Small
- added C39: 56pF, symbol Device:C_Small
- added C40: 10µF, Capacitor_SMD:C_0805_2012Metric, symbol Device:C_Small
- added C41: 4.7µF, Capacitor_SMD:C_0805_2012Metric, symbol Device:C_Small
- added C43, C44: 1µF, Capacitor_SMD:C_0805_2012Metric, symbol Device:C_Small
- added D12, D13, D4, D5 (x2), D8: MBRX120, Adafruit bq25185 Breakout:SOD-123FL, symbol Adafruit bq25185 Breakout-eagle-import:DIODE-SCHOTTKYSOD-123FL
- added D2: BAT54AW, Package_TO_SOT_SMD:SOT-323_SC-70, symbol Diode:BAT54AW
- added D3: BZV55B5V1, Diode_SMD:D_MiniMELF, symbol Diode:BZV55B5V1
- added F3: Polyfuse, LIB_MINISMDC110F-2:MINISMDC050F2, symbol Device:Polyfuse
- added J1, J13, J14, J15: Conn_01x02, Connector_PinSocket_2.54mm:PinSocket_1x02_P2.54mm_Vertical, symbol Connector_Generic:Conn_01x02
- added J10: 732511150, CONN_73251-1150_MOL, symbol CONN_73251-1150_MOL:732511150
- added J11, J12: Conn_01x02, symbol Connector_Generic:Conn_01x02
- added J9: Conn_01x08, symbol Connector_Generic:Conn_01x08
- added JP1, JP3, JP4, JP7: SolderJumper_2_Bridged, Jumper:SolderJumper-2_P1.3mm_Bridged_RoundedPad1.0x1.5mm, symbol Jumper:SolderJumper_2_Bridged
- added L2: 27nH, symbol Device:L_Small
- added Q4: 2N7002, Package_TO_SOT_SMD:SOT-23, symbol Transistor_FET:2N7002
- added R24, R28, R29, R33: 100K, Resistor_SMD:R_0805_2012Metric, symbol Device:R_Small
- added R25, R30, R33, R57: 1M, Resistor_SMD:R_0805_2012Metric, symbol Device:R_Small
- added R26, R35, R39, R58: 100k, Resistor_SMD:R_0805_2012Metric, symbol Device:R_Small
- added R27: 147K, Resistor_SMD:R_0805_2012Metric, symbol Device:R_Small
- added R31: 105K, Resistor_SMD:R_0805_2012Metric, symbol Device:R_Small
- added R34: 1k, Resistor_SMD:R_0805_2012Metric, symbol Device:R_Small
- added R36, R55: NC, Resistor_SMD:R_0805_2012Metric, symbol Device:R_Small
- added R40: 267K, Resistor_SMD:R_0805_2012Metric, symbol Device:R_Small
- added S4, S5, S6: PTS815_SJM_250_SMTR_LFS, PTS815_SJM_250_SMTR_LFS:PTS815SJM250SMTRLFS, symbol SoundRecorder_2.0:PTS815_SJM_250_SMTR_LFS
- added SW2, SW3: PTS815 SJM 250 SMTR LFS, SW4_PTS815 SJM 250 SMTR LFS_CNK, symbol PTS815:PTS815_SJM_250_SMTR_LFS
- added TP7, TP8: TestPoint, TestPoint:TestPoint_Pad_D1.0mm, symbol Connector:TestPoint
- added U14, U18, U24, U29: AO6604, TSOP6_AOS, symbol ao6604:AO6604
- added U15: LP5907MFX-1.8/NOPB, DBV0005A_N, symbol LP5907MFX:LP5907MFX-1.8_NOPB
- added U17: MAX-M10M-00B, MOD18_MAX-M10M_UBL, symbol MAX-M10N-00B:MAX-M10M-00B
- added U17, U28: TPL5111DDCR, DDC0006A_N, symbol TLP5111:TPL5111DDCR
- added U19, U21: AO3407A, SOT-23-3L_AOS, symbol AO3407A:AO3407A
- added U20, U23: TPL5010QDDCRQ1, DDC6_TEX, symbol TPL5010:TPL5010QDDCRQ1
- added U25: TPS62842DGRR, VSSOP_42DGRR_TEX, symbol TPS62842D:TPS62842DGRR
- C34, J1, JP1, Q1, R20, R34, R35, S1: now not fitted; now left out of the parts list
- R32: value 100K -> 100k; now not fitted; now left out of the parts list
- R37: value 33R -> 1M
- R50: value 33R -> 100K; now not fitted; now left out of the parts list
- R51: value 33R -> 1k; now not fitted; now left out of the parts list
- U11: value TPL5110 -> TPL5111; now not fitted; now left out of the parts list
- renumbered C19 to C1, C13 to C10, C12 to C11, C14 to C12, C23 to C13, C25 to C14, C24 to C15, C26 to C16, C1 to C17, C2 to C18, C3 to C19, C21 to C2, C4 to C20, C5 to C21, C6 to C22, C7 to C23, C8 to C24, C9 to C25, C10 to C26, C41 to C27, C40 to C28, C20 to C3, C35 to C34, C36 to C35, C22 to C4, C15 to C5, C17 to C6, C16 to C7, C18 to C8, C11 to C9, D3 to D1, J9 to J2, J10 to J3, J7 to J4, J2 to J5, J8 to J6, J4 to J7, J11 to J8, R10 to R1, R4 to R10, R3 to R11, R5 to R12, R14 to R13, R16 to R14, R17 to R16, R1 to R17, R39 to R18, R41 to R19, R12 to R2, R40 to R20, R53 to R21, R52 to R22, R54 to R23, R56 to R24, R59 to R25, R60 to R26, R21 to R27, R11 to R3, R36 to R38, R13 to R4, R6 to R5, R8 to R6, R9 to R8, R2 to R9, U6 to U1, U13 to U10, U14 to U12, U15 to U13, U12 to U19, U7 to U2, U4 to U3, U5 to U4, U2 to U5, U3 to U6, U8 to U7, U9 to U8, U1 to U9
Connections:
- net +1V8: now also C44.1, TP8.1, U15.5 (VOUT); no longer TP2.1
- net +3.3V: now also C43.2, TP7.1, U15.1 (VIN), U15.3 (EN); no longer TP1.1
- net +5V: now also F3.1
- net BCLK_TDM1_3.3V: now also U10.21 (29_TX7)
- net BCLK_TDM2_3.3V: now also U10.4 (2_OUT2); no longer R50.1
- net Done: now also R37.1, R25.1, R33.1, R57.1, U17.4 (DONE), U20.4 (DONE), U23.4 (DONE), U28.4 (DONE)
- net FSYNC_TDM1_3.3V: now also U10.20 (28_RX7)
- net FSYNC_TDM2_3.3V: now also U10.3 (1_TX1_CTX2_MISO1); no longer R51.1
- net GND: now also R37.2, R50.2, TP2.1, U13.11 (EPAD), C31.2, C32.2, C32.2, C33.1, C33.1, C40.2, C41.2, C43.1, C44.2, C46.2, C47.1, J10.2, J10.3, J11.2 (Pin_2), J12.2 (Pin_2), Q4.2 (S), R24.2, R25.2, R27.2, R29.2, R31.2, R33.2, R33.2, R40.2, R57.2, SW3.3, U14.5 (S1), U15.2 (GND), U17.1 (GND), U17.10 (GND), U17.12 (GND), U17.2 (GND), U18.5 (S1), U20.2 (GND), U23.2 (GND), U24.5 (S1), U25.3 (MODE), U25.8 (GND), U25.EPAD, U28.2 (GND), U29.5 (S1)
- net MCLK_TDM1_3.3V: now also U10.23 (31_CTX3)
- net MCLK_TDM2_3.3V: now also U10.33 (41_A17)
- net OUTPUT_TDM1_3.3V: now also U10.8 (6_OUT1D); no longer R37.1
- net OUTPUT_TDM2_3.3V: now also U10.5 (3_LRCLK2)
- net PWR: now also J1.1 (Pin_1), J13.1 (Pin_1), J14.1 (Pin_1), J15.1 (Pin_1), JP1.2 (B), JP3.2 (B), JP4.2 (B), JP7.2 (B)
- net RXGPS: now also U10.26 (34_RX8), J9.5 (Pin_5), U17.3 (RXD)
- net SENSORSDA: now also U10.17 (25_A11_RX6_SDA2)
- net SHDNZ_1.8V: now also U19.9 (A8)
- net TXGPS: now also U10.27 (35_TX8), J9.4 (Pin_4), U17.2 (TXD)
- net VBAT: now also J11.1 (Pin_1); no longer U10.50 (VBAT), U12.1, U12.2
- net VBUS: now also J12.1 (Pin_1)
- net battery voltage: now also U10.18 (26_A12_MOSI1), R30.2, R31.1; no longer U10.17 (25_A11_RX6_SDA2)
- net emrg_pwr_swch: now also R29.1, U14.1 (G1)
- net sensorSCL: now also U10.16 (24_A10_TX6_SCL2)
- net at C34.1, Q1.4 (SOURCE), R20.1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: no longer L1.2
- net GPS_PWR: now reaches U10.15 (3V3)
- net GPS_PWR: now also J9.1 (Pin_1), J9.8 (Pin_8), R39.1, U21.2 (S)
- net SLEEP_LATCH: now reaches U10.22 (30_CRX3)
- net SLEEP_LATCH: now also D13.A, D5.A
- net at R51.2: now also C47.2, U29.1 (G1); no longer U10.3 (1_TX1_CTX2_MISO1)
- net GPS_ON: now reaches U10.31 (39_MISO1_OUT1A)
- net GPS_ON: now also J9.2 (Pin_2), J9.7 (Pin_7), R39.2, U21.1 (G)
- net at U10.45 (23_A9_CRX1_MCLK1): now also SW3.1
- net at R32.2: now also U24.3 (G2), U24.6 (D1)
- net at U13.7 (ILIM/VSET): now also D3.1 (K); no longer SW1.2 (B)
- net CAPACITOR: now reaches Q1.3 (GATE), R20.2, U11.5 (DRV)
- net at L1.1: now also U25.2 (SW)
- net at R32.1: now also C32.1, S5.1 (COM_1), U23.1 (VDD), U24.2 (S2)
- new net: U17.7 (V_IO), U17.8 (VCC), U21.3 (D)
- new net: C32.1, C40.1, L1.2, SW2.1, U17.1 (VDD), U17.6 (EN_ONE_SHOT), U18.2 (S2), U25.1 (VOS)
- new net: R33.1, SW2.3, U17.3 (DELAY_M_DRV)
- new net: C41.1, F3.2, R28.1, TP1.1, U14.2 (S2), U25.5 (EN), U25.6 (VIN)
- new net: R58.1, U29.3 (G2)
- new net: R58.2, U29.6 (D1)
- new net: D2.2, U10.50 (VBAT)
- new net: D4.C, D5.C, R34.1
- new net: C33.2, R34.2, U18.1 (G1)
- new net: D12.A, R55.1
- new net: R55.2, U28.5 (DRV)
- new net: R28.2, U14.3 (G2), U14.6 (D1)
- new net: R30.1, U14.4 (D2)
- new net: D3.2 (A), SW1.2 (B)
- new net: R35.1, U18.3 (G2)
- new net: R35.2, U18.6 (D1)
- new net: C31.1, Q4.3 (D), R26.2, S4.1 (COM_1), U19.2 (S), U20.1 (VDD)
- new net: R24.1, S4.3 (NO_1), U20.3 (DELAY/M_RST)
- new net: Q4.1 (G), U20.5 (WAKE)
- new net: C39.1, U17.11 (RF_IN)
- new net: J15.2 (Pin_2), JP7.1 (A), U29.4 (D2)
- new net: C33.2, D5.C, D8.C, U24.1 (G1)
- new net: J14.2 (Pin_2), JP4.1 (A), U24.4 (D2)
- new net: R26.1, U19.1 (G)
- new net: J13.2 (Pin_2), JP3.1 (A), U19.3 (D)
- new net: C46.1, S6.1 (COM_1), U28.1 (VDD), U28.6 (EN_ONE_SHOT), U29.2 (S2)
- new net: R50.1, S6.3 (NO_1), U28.3 (DELAY_M_DRV)
- new net: L2.1, U17.14 (VCC_RF)
- new net: J1.2 (Pin_2), JP1.1 (A), U18.4 (D2)
- new net: R36.2, U17.5 (DRV)
- new net: D12.C, D13.C, R51.1
- new net: D4.A, R36.1
- new net: R27.1, S5.3 (NO_1), U23.3 (DELAY/M_RST)
- new net: R40.1, U25.4 (VSET)
- new net: D8.A, U23.5 (WAKE)
- new net: D2.3, U12.1, U12.2
- new net GPS_EN: J9.6 (Pin_6)
- new net GPS_RTC: D2.1, U17.6 (V_BCKP)
- new net Latch_PWR: D5.A
- new net TMPPS: J9.3 (Pin_3), U17.4 (TIMEPULSE)
- new net antenna: C39.2, J10.1, L2.2
- no-connect marks 28 -> 67
Other:
- note added: "GNSS (GPS)"
- note added: "GPS"
- note added: "GPS PIN TESTER"
- note added: "GPS antenna conector (has to be in the edge, and close to the gps)"
- note added: "Microphones 1 & 2"
- note added: "Microphones 3 & 4"
- note added: "Microphones 5 & 6"
- note added: "Microphones 7 & 8"
- note added: "SOLUTION 1"
- note added: "SOLUTION 3"
- note added: "SOLUTION 4"
- note added: "SOLUTION2"
- note added: "Sensor port"
- note added: "Solar and battery charging module"
- note added: "Solar in TESTER"
- note added: "analog ground"
- note added: "battery conector (has to be a different pin layout)"
- note added: "step down converter from 1.8 to 5v"
- note removed: "ADD DIODE"
- note removed: "Battery connection"
- note removed: "MAKE ALL CAPACITORSS AND RESITANCE CERAMIC"
- note removed: "Solar panel conector"
- note removed: "TO DO: implement ADAFRUIT change every resistor and capacitor number add every part into the libraries fix lighting"
- note removed: "step down covnerter from 1.8 to 5v"
- moved on the sheet: C17, C18, C19, C20, C21, C22, C23, C24, C25, C26, C34, C35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

Commit message: pcb sketch v1
Parts:
- removed C31, C32, C34, C46: 100nF, Capacitor_SMD:C_0805_2012Metric, symbol Device:C_Small
- removed C33, C47: 1000nF, symbol Device:C_Small
- removed CHG1: ORANGE, Adafruit bq25185 Breakout:CHIPLED_0805_NOOUTLINE, symbol Adafruit bq25185 Breakout-eagle-import:LED0805_NOOUTLINE
- removed D12, D13, D4 (x2), D5 (x2), D8: MBRX120, Adafruit bq25185 Breakout:SOD-123FL, symbol Adafruit bq25185 Breakout-eagle-import:DIODE-SCHOTTKYSOD-123FL
- removed D3: BZV55B5V1, Diode_SMD:D_MiniMELF, symbol Diode:BZV55B5V1
- removed FAULT1: RED, Adafruit bq25185 Breakout:CHIPLED_0805_NOOUTLINE, symbol Adafruit bq25185 Breakout-eagle-import:LED0805_NOOUTLINE
- removed J1, J13, J14, J15: Conn_01x02, Connector_PinSocket_2.54mm:PinSocket_1x02_P2.54mm_Vertical, symbol Connector_Generic:Conn_01x02
- removed J7: Conn_01x09, symbol Connector_Generic:Conn_01x09
- removed JP1, JP3, JP4, JP7: SolderJumper_2_Bridged, Jumper:SolderJumper-2_P1.3mm_Bridged_RoundedPad1.0x1.5mm, symbol Jumper:SolderJumper_2_Bridged
- removed Q1: CPH6350-TL-W, SOT95P280X105-6N, symbol SoundRecorder_2.0:CPH6350-TL-W
- removed Q4: 2N7002, Package_TO_SOT_SMD:SOT-23, symbol Transistor_FET:2N7002
- removed R20, R55: NC, Resistor_SMD:R_0805_2012Metric, symbol Device:R_Small
- removed R24, R34, R50: 100K, Resistor_SMD:R_0805_2012Metric, symbol Device:R_Small
- removed R25, R33, R35, R57: 1M, Resistor_SMD:R_0805_2012Metric, symbol Device:R_Small
- removed R26, R32, R58: 100k, Resistor_SMD:R_0805_2012Metric, symbol Device:R_Small
- removed R27: 147K, Resistor_SMD:R_0805_2012Metric, symbol Device:R_Small
- removed R51: 1k, Resistor_SMD:R_0805_2012Metric, symbol Device:R_Small
- removed S1, S4, S5, S6: PTS815_SJM_250_SMTR_LFS, PTS815_SJM_250_SMTR_LFS:PTS815SJM250SMTRLFS, symbol SoundRecorder_2.0:PTS815_SJM_250_SMTR_LFS
- removed SW1: SW_SPDT, symbol Switch:SW_SPDT
- removed U11: TPL5111, TPL5110DDCR:SOT95P280X110-6N, symbol SoundRecorder_2.0:TPL5110DDCR
- removed U19: AO3407A, SOT-23-3L_AOS, symbol AO3407A:AO3407A
- removed U20, U23: TPL5010QDDCRQ1, DDC6_TEX, symbol TPL5010:TPL5010QDDCRQ1
- removed U24, U29: AO6604, TSOP6_AOS, symbol ao6604:AO6604
- removed U28: TPL5111DDCR, DDC0006A_N, symbol TLP5111:TPL5111DDCR
- added CHG1, Fault1: SFH2701, LED_SMD:LED_1206_3216Metric_Castellated, symbol Sensor_Optical:SFH2701
- added D4, D5, D6: MBRX120LF-TP, MBRX120LF:SOD3716X135N, symbol MBRX120LF:MBRX120LF-TP
- added D7: BZV55B5V1, Diode_SMD:D_MiniMELF, symbol Diode:BZV55B5V1
- added S2: SLW-12689-4A-N-D, SLW12689:SLW126894AND, symbol switch:SLW-12689-4A-N-D
- BAT1: renamed from U12; footprint LIB_3034:BatteryHolder_Keystone_3034_1x20mm -> 79523211:79523211
- C33, C39: footprint (none) -> Capacitor_SMD:C_0201_0603Metric
- D1: footprint APHF1608LSEEQBDZGKC-2:LED_APHF1608LSEEQBDZGKC -> LED_SMD:LED-APA102-2020
- F3: footprint LIB_MINISMDC110F-2:MINISMDC050F2 -> MINISMDC050F-2:MINISMDC050F2
- J1: footprint Connector_PinSocket_2.54mm:PinSocket_1x02_P2.54mm_Vertical -> Connector_PinHeader_1.00mm:PinHeader_1x02_P1.00mm_Horizontal
- J10: footprint CONN_73251-1150_MOL -> DFE201612E:1286ASH1R0MP2
- J11: renamed from J12; footprint (none) -> Connector_PinHeader_1.00mm:PinHeader_1x02_P1.00mm_Horizontal
- J12: renamed from J11; footprint (none) -> Connector_PinHeader_1.00mm:PinHeader_1x02_P1.00mm_Horizontal
- J2, J3: footprint (none) -> RJHSE-3380:CONN_RJHSE-3380_AMP
- J4, J6: footprint (none) -> Connector_PinHeader_1.00mm:PinHeader_1x07_P1.00mm_Horizontal
- J5: footprint Connector_PinSocket_2.54mm:PinSocket_1x04_P2.54mm_Vertical -> Connector_PinHeader_1.00mm:PinHeader_1x04_P1.00mm_Horizontal
- J7: renamed from J8; footprint (none) -> Connector_PinHeader_1.00mm:PinHeader_1x04_P1.00mm_Horizontal
- J8: renamed from J9; footprint (none) -> Connector_PinHeader_1.00mm:PinHeader_1x08_P1.00mm_Horizontal
- J9: renamed from J6; footprint (none) -> 10118192:101181920002LF
- L1: footprint 1286ASH1R0MP2 -> DFE201612E:1286ASH1R0MP2
- L2: footprint (none) -> LQM2HPZ2R2MG0L:LQM2HPN1R0MG0L
- R21, R22, R23, R24, R27: footprint Adafruit bq25185 Breakout:0603-NO -> Resistor_SMD:R_0805_2012Metric
- R25: value 5.1K -> 6.8K; footprint Adafruit bq25185 Breakout:0603-NO -> Resistor_SMD:R_0805_2012Metric
- R26: value 6.8K -> 5.1K; footprint Adafruit bq25185 Breakout:0603-NO -> Resistor_SMD:R_0805_2012Metric
- SW2, SW3: footprint SW4_PTS815 SJM 250 SMTR LFS_CNK -> PTS815:SW4_PTS815 SJM 250 SMTR LFS_CNK
- U1, U2, U3, U4, U5, U6, U7, U8: footprint IM66D132H:IFX-PG-TLGA-5N-9-V -> mics:IFX-PG-TLGA-5N-9-V
- U10: footprint (none) -> Teensy:Teensy41
- U11: renamed from U13; footprint WSON10_DLH_TEX -> BQ25185DLHR:BQ25185DLHR
- U12: renamed from U14; footprint TSOP6_AOS -> AO6604:AO6604
- U13: renamed from U25; footprint VSSOP_42DGRR_TEX -> TPS6284:TPS62842DGRR
- U14: renamed from U17; footprint DDC0006A_N -> TPL5111DDCR:TPL5111DDCR
- U15: renamed from U18; footprint TSOP6_AOS -> AO6604:AO6604
- U17: renamed from U15; footprint DBV0005A_N -> ul_LP5907MFX-1-2-NOPB:DBV0005A_N
- U18: renamed from U21; footprint SOT-23-3L_AOS -> AO3407A:SOT-23-3L_AOS
- U19: renamed from U17; footprint MOD18_MAX-M10M_UBL -> MAX-M10M:MAX-M10M-00B
- renumbered U19 to U16
Connections:
- net +5V: now also CHG1.2 (A), Fault1.2 (A)
- net GND: now also R25.1, R26.1, S2.4 (MH1), S2.5 (MH2); no longer R25.2, R26.2
- net SLEEP_LATCH: now also D5.2 (A)
- net VBUS: now also D6.1 (K)
- net at R21.2: now also CHG1.1 (K)
- net at R34.1: now also D4.1 (K), D5.1 (K)
- net at U11.7 (ILIM/VSET): now also D7.1 (K)
- net at R36.1: now also D4.2 (A)
- net at J9.1 (VBUS): now also D6.2 (A)
- net at R23.2: now also Fault1.1 (K)
- new net: R25.2, S2.1
- new net: R26.2, S2.3
- new net: D7.2 (A), S2.2
- no-connect marks 67 -> 56
Other:
- note removed: "ADD CAPACITOR FOR MAINTAINING THE BOARD ON"
- note removed: "PCMD3180 and timer testing port"
- note removed: "SOLUTION 1"
- note removed: "SOLUTION 3"
- note removed: "SOLUTION 4"
- note removed: "SOLUTION2"
- moved on the sheet: C38, J10, J11, J12, J3, J4, J5, J7, J8, J9, R34, R36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

Commit message: pcb savepoint
Parts:
- CHG1, Fault1: footprint LED_SMD:LED_1206_3216Metric_Castellated -> LED_SMD:LED-APA102-2020
- J10: footprint DFE201612E:1286ASH1R0MP2 -> 73251:CONN_73251-1150_MOL
- U14: footprint TPL5111DDCR:TPL5111DDCR -> TPL5111DDCR:DDC0006A_L
Changed lines of the file:
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@@
 			)
 		)
-		(property "Footprint" "LED_SMD:LED_1206_3216Metric_Castellated"
+		(property "Footprint" "LED_SMD:LED-APA102-2020"
 			(at 109.22 164.465 0)
 			(effects
@@
 			)
 		)
-		(property "Footprint" "LED_SMD:LED_1206_3216Metric_Castellated"
+		(property "Footprint" "LED_SMD:LED-APA102-2020"
 			(at 25.4 183.515 0)
 			(effects
@@
 			)
 		)
-		(property "Footprint" "DFE201612E:1286ASH1R0MP2"
+		(property "Footprint" "73251:CONN_73251-1150_MOL"
 			(at 547.37 241.3 0)
 			(effects
@@
 			)
 		)
-		(property "Footprint" "TPL5111DDCR:TPL5111DDCR"
+		(property "Footprint" "TPL5111DDCR:DDC0006A_L"
 			(at 232.41 248.92 0)
 			(effects
