File: Hardware/SongBeam 3.1_kicad/SongBeam4.0/SongBeam4.0.kicad_sch (KiCad schematic)
At the start: 129 parts, among them J1 Conn_01x02, J10 732511150, J11 Conn_01x02, J12 Conn_01x02, J2 RJ45, J3 RJ45, J4 Conn_01x07, J5 Conn_01x04, J6 Conn_01x07, J7 Conn_01x04, J8 Conn_01x08, J9 USB_B_Micro, SW2 PTS815 SJM 250 SMTR LFS, SW3 PTS815 SJM 250 SMTR LFS, U1 IM66D132H, U10 Teensy4.1, U11 BQ25185DLHR, U12 AO6604, U13 TPS62842DGRR, U14 TPL5111DDCR, U15 AO6604, U16 TXS0108EPW, U17 LP5907MFX-1.8/NOPB, U18 AO3407A, U19 MAX-M10M-00B, U2 IM66D132H, U3 IM66D132H, U4 IM66D132H, U5 IM66D132H, U6 IM66D132H, U7 IM66D132H, U8 IM66D132H, U9 PCMD3180IRTWR

Commit message: prerouting
Parts:
- removed CHG1, Fault1: SFH2701, LED_SMD:LED-APA102-2020, symbol Sensor_Optical:SFH2701
- added CHG1, FAULT1: SFH_2716_A01, LEDSB:LEDC2012X100N, symbol ledsSB:SFH_2716_A01
- J1, J11, J12: footprint Connector_PinHeader_1.00mm:PinHeader_1x02_P1.00mm_Horizontal -> Connector_PinHeader_1.00mm:PinHeader_1x02_P1.00mm_Vertical
- J4, J6: footprint Connector_PinHeader_1.00mm:PinHeader_1x07_P1.00mm_Horizontal -> Connector_PinHeader_1.00mm:PinHeader_1x07_P1.00mm_Vertical
- J5, J7: footprint Connector_PinHeader_1.00mm:PinHeader_1x04_P1.00mm_Horizontal -> Connector_PinHeader_1.00mm:PinHeader_1x04_P1.00mm_Vertical
- J8: footprint Connector_PinHeader_1.00mm:PinHeader_1x08_P1.00mm_Horizontal -> Connector_PinHeader_1.00mm:PinHeader_1x08_P1.00mm_Vertical
Connections:
- net +5V: now also CHG1.2 (A), FAULT1.2 (A)
- net at R21.2: now also CHG1.1 (K)
- net at R23.2: now also FAULT1.1 (K)
Other:
- moved on the sheet: C29

Commit message: Pcb bugfixxing
Parts:
- removed R21, R23: 1K, Resistor_SMD:R_0805_2012Metric, symbol Adafruit bq25185 Breakout-eagle-import:RESISTOR_0603_NOOUT
- removed R22, R27: 10K, Resistor_SMD:R_0805_2012Metric, symbol Adafruit bq25185 Breakout-eagle-import:RESISTOR_0603_NOOUT
- removed R24: 300, Resistor_SMD:R_0805_2012Metric, symbol Adafruit bq25185 Breakout-eagle-import:RESISTOR_0603_NOOUT
- removed R25: 6.8K, Resistor_SMD:R_0805_2012Metric, symbol Adafruit bq25185 Breakout-eagle-import:RESISTOR_0603_NOOUT
- removed R26: 5.1K, Resistor_SMD:R_0805_2012Metric, symbol Adafruit bq25185 Breakout-eagle-import:RESISTOR_0603_NOOUT
- added R21, R23: 1K, Resistor_SMD:R_0805_2012Metric, symbol Device:R_Small
- added R22: 10K, Resistor_SMD:R_0805_2012Metric, symbol Device:R_Small
- added R24: 300, Resistor_SMD:R_0805_2012Metric, symbol Device:R_Small
- added R25: 6.8k, Resistor_SMD:R_0805_2012Metric, symbol Device:R_Small
- added R26: 5.1k, Resistor_SMD:R_0805_2012Metric, symbol Device:R_Small
- added R27: 10k, Resistor_SMD:R_0805_2012Metric, symbol Device:R_Small
- U14: footprint TPL5111DDCR:DDC0006A_L -> TPL5111DDCR:SOT95P280X110-6N
Connections:
- net GND: now also R22.2, R24.2, R25.2, R26.2, R27.1
- net at U11.3 (STAT2): now also R21.1
- net at CHG1.1 (K): now also R21.2
- net at U11.8 (ISET): now also R24.1
- net at U11.4 (/CE): now also R22.1
- net at U11.6 (TS/MR): now also R27.2
- net at U11.9 (STAT1): now also R23.2
- net at S2.1: now also R25.1
- net at FAULT1.1 (K): now also R23.1
- net at S2.3: now also R26.1

Commit message: debugging
Connections:
- net TestGRP1 is gone; now on net testGRP1: R1.1, U1.1 (DATA)
Changed lines of the file:
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@@
 		)
 	)
-	(global_label "TestGRP1"
+	(global_label "testGRP1"
 		(shape input)
 		(at 54.61 50.8 180)
@@
 		)
 		(property "Intersheetrefs" "${INTERSHEET_REFS}"
-			(at 42.7953 50.8 0)
+			(at 43.0372 50.8 0)
 			(effects
 				(font

Commit message: Layout updates
Parts:
- removed D4: MBRX120LF-TP, MBRX120LF:SOD3716X135N, symbol MBRX120LF:MBRX120LF-TP
- removed L2: 27nH, LQM2HPZ2R2MG0L:LQM2HPN1R0MG0L, symbol Device:L_Small
- removed R36: NC, Resistor_SMD:R_0805_2012Metric, symbol Device:R_Small
- added C30: 10nF, Capacitor_SMD:C_0201_0603Metric, symbol Device:C_Small
- added D8: MBRX120LF-TP, MBRX120LF:SOD3716X135N, symbol MBRX120LF:MBRX120LF-TP
- added L2: GJM1555C1H470JB01D, GPSINDUCTOR:CAPC1005X55N, symbol inductor GPS:GJM1555C1H470JB01D
- C29: value 1uF -> 22uF
- C33: value 1000nF -> 100muF
- C39: value 56pF -> 47pF
Connections:
- net GND: now also C33.2, C30.2; no longer C33.1
- net PWR: now also C33.1
- net TMPPS: now also U10.7 (5_IN2)
- net VBUS: now also D8.1 (K); no longer J11.1 (Pin_1)
- net antenna: now also L2.2
- net at D5.1 (K), R34.1: now also U14.5 (DRV)
- net at R34.2, U15.1 (G1): no longer C33.2
- net at U19.14 (VCC_RF): now also C30.1, L2.1
- new net: D8.2 (A), J11.1 (Pin_1)
- no-connect marks 56 -> 55
Other:
- moved on the sheet: C33
