File: Hardware/Daughterboard_A/daugtherboard_1.1.kicad_pcb (KiCad board)
At the start: 2 copper layers, 165.6 x 82.3 mm, 72 parts, among them J2 RJ45, J3 RJ45, J4 Conn_01x07, J5 Conn_01x04, J6 Conn_01x07, U1 IM66D132H, U16 TXS0108EPW, U17 LP5907MFX-1.8/NOPB, U2 IM66D132H, U3 IM66D132H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

Commit message: 4.1
Parts:
- R2: value 100R -> 100K
