File: Hardware/Daughterboard_A/daugtherboard_1.1.kicad_sch (KiCad schematic)
At the start: 66 parts, among them J2 RJ45, J3 RJ45, J4 Conn_01x07, J5 Conn_01x04, J6 Conn_01x07, U1 IM66D132H, U16 TXS0108EPW, U17 LP5907MFX-1.8/NOPB, U2 IM66D132H, U3 IM66D132H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

Commit message: 4.1
Parts:
- R2: value 100R -> 100K
Changed lines of the file:
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@@
 	)
 	(junction
-		(at 157.48 36.83)
-		(diameter 0)
-		(color 0 0 0 0)
-	)
-	(junction
 		(at 312.42 26.67)
 		(diameter 0)
@@
 	)
 	(junction
-		(at 153.67 187.96)
+		(at 31.75 26.67)
 		(diameter 0)
 		(color 0 0 0 0)
 	)
 	(junction
-		(at 33.02 100.33)
+		(at 153.67 187.96)
 		(diameter 0)
 		(color 0 0 0 0)
@@
 	)
 	(junction
-		(at 33.02 26.67)
-		(diameter 0)
-		(color 0 0 0 0)
-	)
-	(junction
 		(at 189.23 177.8)
 		(diameter 0)
@@
 	)
 	(junction
-		(at 157.48 100.33)
-		(diameter 0)
-		(color 0 0 0 0)
-	)
-	(junction
 		(at 323.85 34.29)
 		(diameter 0)
@@
 		(color 0 0 0 0)
 	)
-	(junction
-		(at 33.02 36.83)
-		(diameter 0)
-		(color 0 0 0 0)
-	)
 	(no_connect
 		(at 83.82 185.42)
@@
 	(wire
 		(pts
-			(xy 27.94 26.67) (xy 33.02 26.67)
+			(xy 27.94 26.67) (xy 31.75 26.67)
 		)
 		(stroke
@@
 	(wire
 		(pts
-			(xy 157.48 26.67) (xy 157.48 36.83)
-		)
-		(stroke
-			(width 0)
-			(type default)
-		)
-	)
-	(wire
-		(pts
 			(xy 247.65 119.38) (xy 251.46 119.38)
 		)
@@
 	(wire
 		(pts
-			(xy 33.02 90.17) (xy 33.02 100.33)
+			(xy 33.02 90.17) (xy 33.02 105.41)
 		)
 		(stroke
@@
 	(wire
 		(pts
-			(xy 33.02 36.83) (xy 33.02 41.91)
+			(xy 31.75 26.67) (xy 31.75 41.91)
 		)
 		(stroke
@@
 	(wire
 		(pts
+			(xy 31.75 41.91) (xy 33.02 41.91)
+		)
+		(stroke
+			(width 0)
+			(type default)
+		)
+	)
+	(wire
+		(pts
 			(xy 152.4 26.67) (xy 157.48 26.67)
 		)
@@
 	(wire
 		(pts
+			(xy 27.94 36.83) (xy 33.02 36.83)
+		)
+		(stroke
+			(width 0)
+			(type default)
+		)
+	)
+	(wire
+		(pts
 			(xy 187.96 110.49) (xy 195.58 110.49)
 		)
@@
 	(wire
 		(pts
-			(xy 33.02 26.67) (xy 33.02 36.83)
-		)
-		(stroke
-			(width 0)
-			(type default)
-		)
-	)
-	(wire
-		(pts
 			(xy 262.89 58.42) (xy 262.89 62.23)
 		)
@@
 	(wire
 		(pts
-			(xy 157.48 36.83) (xy 157.48 41.91)
+			(xy 157.48 26.67) (xy 157.48 41.91)
 		)
 		(stroke
@@
 	(wire
 		(pts
-			(xy 157.48 90.17) (xy 157.48 100.33)
+			(xy 157.48 90.17) (xy 157.48 105.41)
 		)
 		(stroke
@@
 	(wire
 		(pts
-			(xy 157.48 100.33) (xy 157.48 105.41)
-		)
-		(stroke
-			(width 0)
-			(type default)
-		)
-	)
-	(wire
-		(pts
 			(xy 27.94 90.17) (xy 33.02 90.17)
 		)
@@
 	(wire
 		(pts
-			(xy 33.02 26.67) (xy 71.12 26.67)
-		)
-		(stroke
-			(width 0)
-			(type default)
-		)
-	)
-	(wire
-		(pts
 			(xy 341.63 26.67) (xy 341.63 35.56)
 		)
@@
 	(wire
 		(pts
-			(xy 33.02 100.33) (xy 33.02 105.41)
+			(xy 259.08 176.53) (xy 259.08 180.34)
 		)
 		(stroke
-			(width 0)
+			(width 0.2)
 			(type default)
+			(color 128 77 0 1)
 		)
 	)
 	(wire
 		(pts
-			(xy 259.08 176.53) (xy 259.08 180.34)
+			(xy 59.69 52.07) (xy 59.69 48.26)
 		)
 		(stroke
-			(width 0.2)
+			(width 0)
 			(type default)
-			(color 128 77 0 1)
 		)
 	)
 	(wire
 		(pts
-			(xy 59.69 52.07) (xy 59.69 48.26)
+			(xy 31.75 26.67) (xy 71.12 26.67)
 		)
 		(stroke
@@
 	(wire
 		(pts
-			(xy 27.94 36.83) (xy 33.02 36.83)
-		)
-		(stroke
-			(width 0)
-			(type default)
-		)
-	)
-	(wire
-		(pts
 			(xy 195.58 90.17) (xy 201.93 90.17)
 		)
@@
 			)
 		)
-		(property "Value" "100R"
-			(at 61.722 61.976 0)
+		(property "Value" "100K"
+			(at 61.976 61.722 0)
 			(effects
 				(font

Commit message: 4.1.1
Connections:
- net GND: now also J3.1, J3.2
- no-connect marks 5 -> 3
Changed lines of the file:
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@@
 	)
 	(no_connect
-		(at 83.82 185.42)
-	)
-	(no_connect
-		(at 83.82 182.88)
-	)
-	(no_connect
 		(at 328.93 53.34)
 	)
@@
 	)
 	(symbol
+		(lib_name "GND_8")
+		(lib_id "power:GND")
+		(at 83.82 182.88 90)
+		(unit 1)
+		(exclude_from_sim no)
+		(in_bom yes)
+		(on_board yes)
+		(dnp no)
+		(property "Reference" "#PWR02"
+			(at 90.17 182.88 0)
+			(effects
+				(font
+					(size 1.27 1.27)
+				)
+				(hide yes)
+			)
+		)
+		(property "Value" "GND"
+			(at 91.948 182.626 90)
+			(effects
+				(font
+					(size 1.27 1.27)
+				)
+				(justify left)
+			)
+		)
+		(property "Footprint" ""
+			(at 83.82 182.88 0)
+			(effects
+				(font
+					(size 1.27 1.27)
+				)
+				(hide yes)
+			)
+		)
+		(property "Datasheet" ""
+			(at 83.82 182.88 0)
+			(effects
+				(font
+					(size 1.27 1.27)
+				)
+				(hide yes)
+			)
+		)
+		(property "Description" "Power symbol creates a global label with name \"GND\" , ground"
+			(at 83.82 182.88 0)
+			(effects
+				(font
+					(size 1.27 1.27)
+				)
+				(hide yes)
+			)
+		)
+		(pin "1"
+		)
+		(instances
+			(project "daugtherboard_1.1"
+				(path "/20cc9ad0-b159-4b68-8c55-e2948c23be5b"
+					(reference "#PWR02")
+					(unit 1)
+				)
+			)
+		)
+	)
+	(symbol
 		(lib_id "Device:C_Small")
 		(at 312.42 30.48 0)
@@
 					(unit 1)
 				)
+			)
+		)
+	)
+	(symbol
+		(lib_name "GND_8")
+		(lib_id "power:GND")
+		(at 83.82 185.42 90)
+		(unit 1)
+		(exclude_from_sim no)
+		(in_bom yes)
+		(on_board yes)
+		(dnp no)
+		(property "Reference" "#PWR03"
+			(at 90.17 185.42 0)
+			(effects
+				(font
+					(size 1.27 1.27)
+				)
+				(hide yes)
+			)
+		)
+		(property "Value" "GND"
+			(at 91.948 185.166 90)
+			(effects
+				(font
+					(size 1.27 1.27)
+				)
+				(justify left)
+			)
+		)
+		(property "Footprint" ""
+			(at 83.82 185.42 0)
+			(effects
+				(font
+					(size 1.27 1.27)
+				)
+				(hide yes)
+			)
+		)
+		(property "Datasheet" ""
+			(at 83.82 185.42 0)
+			(effects
+				(font
+					(size 1.27 1.27)
+				)
+				(hide yes)
+			)
+		)
+		(property "Description" "Power symbol creates a global label with name \"GND\" , ground"
+			(at 83.82 185.42 0)
+			(effects
+				(font
+					(size 1.27 1.27)
+				)
+				(hide yes)
+			)
+		)
+		(pin "1"
+		)
+		(instances
+			(project "daugtherboard_1.1"
+				(path "/20cc9ad0-b159-4b68-8c55-e2948c23be5b"
+					(reference "#PWR03")
+					(unit 1)
+				)
