File: Hardware/SongBeam4.0/SongBeam4.0.kicad_pcb (KiCad board)
At the start: 2 copper layers, 176.9 x 110 mm, 135 parts, among them J1 Conn_01x02, J10 732511150, J11 Conn_01x02, J12 Conn_01x02, J13 Conn_01x01, J2 RJ45, J3 RJ45, J4 Conn_01x07, J5 Conn_01x04, J6 Conn_01x07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

Commit message: change resistor 300 to 300R
Parts:
- R24: value 300 -> 300R
Changed lines of the file:
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@@
 			)
 		)
-		(property "Value" "300"
+		(property "Value" "300R"
 			(at 0 1.65 90)
 			(layer "F.Fab")
