File: Hardware/SongBeam4.0/SongBeam4.0.kicad_pcb (KiCad board)
At the start: 2 copper layers, 176.9 x 110 mm, 135 parts, among them J1 Conn_01x02, J10 732511150, J11 Conn_01x02, J12 Conn_01x02, J13 Conn_01x01, J2 RJ45, J3 RJ45, J4 Conn_01x07, J5 Conn_01x04, J6 Conn_01x07, J7 Conn_01x04, J8 Conn_01x06, J9 USB_B_Micro, Q2 DTC143ZEBTL, SW2 PTS815 SJM 250 SMTR LFS, SW3 PTS815 SJM 250 SMTR LFS, U1 IM66D132H, U10 Teensy4.1, U11 BQ25185DLHR, U12 AO6604, U13 TPS62842DGRR, U14 TPL5111DDCR, U15 AO6604, U16 TXS0108EPW, U17 LP5907MFX-1.8/NOPB, U19 L86-M33, U2 IM66D132H, U20 AO3407A, U3 IM66D132H, U4 IM66D132H, U5 IM66D132H, U7 IM66D132H, U8 IM66D132H, U9 PCMD3180IRTWR

Commit message: fixed weird bug that keeps deleting microphone
Parts:
- added C11: 100nF, Capacitor_SMD:C_0805_2012Metric, F.Cu at (99.0, 64.8)
- added C12: 47pF, Capacitor_SMD:C_0805_2012Metric, F.Cu at (104.0, 70.1)
- added R11: 100R, Resistor_SMD:R_0805_2012Metric, F.Cu at (100.2, 67.7)
- added U6: IM66D132H, mics:IFX-PG-TLGA-5N-9-V, F.Cu at (102.8, 64.4)
- moved R12 0.41 mm to (104.0, 67.7)
- renumbered ANT_DBG to CHG2
