File: Hardware/SongBeam4.0/SongBeam4.0_BRKOUT.kicad_sch (KiCad schematic)
At the start: 129 parts, among them J1 Conn_01x02, J10 732511150, J11 Conn_01x02, J12 Conn_01x02, J2 RJ45, J3 RJ45, J4 Conn_01x07, J5 Conn_01x04, J6 Conn_01x07, J7 Conn_01x04, J8 Conn_01x08, J9 USB_B_Micro, SW2 PTS815 SJM 250 SMTR LFS, SW3 PTS815 SJM 250 SMTR LFS, U1 IM66D132H, U10 Teensy4.1, U11 BQ25185DLHR, U12 AO6604, U13 TPS62842DGRR, U14 TPL5111DDCR, U15 AO6604, U16 TXS0108EPW, U17 LP5907MFX-1.8/NOPB, U18 AO3407A, U19 MAX-M10M-00B, U2 IM66D132H, U3 IM66D132H, U4 IM66D132H, U5 IM66D132H, U6 IM66D132H, U7 IM66D132H, U8 IM66D132H, U9 PCMD3180IRTWR

Commit message: 4.1.1
Parts:
- removed C30: 10nF, Capacitor_SMD:C_0201_0603Metric, symbol Device:C_Small
- removed C33: 100muF, Capacitor_SMD:C_0201_0603Metric, symbol Device:C_Small
- removed C39: 47pF, Capacitor_SMD:C_0201_0603Metric, symbol Device:C_Small
- removed D7: BZV55B5V1, Diode_SMD:D_MiniMELF, symbol Diode:BZV55B5V1
- removed J8: Conn_01x08, Connector_PinHeader_1.00mm:PinHeader_1x08_P1.00mm_Vertical, symbol Connector_Generic:Conn_01x08
- removed L2: GJM1555C1H470JB01D, GPSINDUCTOR:CAPC1005X55N, symbol inductor GPS:GJM1555C1H470JB01D
- removed R39: 100k, Resistor_SMD:R_0805_2012Metric, symbol Device:R_Small
- removed U18: AO3407A, AO3407A:SOT-23-3L_AOS, symbol AO3407A:AO3407A
- removed U19: MAX-M10M-00B, MAX-M10M:MAX-M10M-00B, symbol MAX-M10N-00B:MAX-M10M-00B
- added C37: 100nf, Capacitor_SMD:C_0805_2012Metric, symbol Device:C_Small
- added C42: 4.7uF, Capacitor_SMD:C_0805_2012Metric, symbol Device:C_Small
- added C45: 100nF, Capacitor_SMD:C_0805_2012Metric, symbol Device:C_Small
- added CHG2: SFH_2716_A01, LEDSB:LEDC2012X100N, symbol ledsSB:SFH_2716_A01
- added H1, H2, H3, H4, H5, H6: 3.2mm, MountingHole:MountingHole_3.2mm_M3_ISO14580, symbol Mechanical:MountingHole
- added J13: Conn_01x01, Connector_PinHeader_1.00mm:PinHeader_1x01_P1.00mm_Vertical, symbol Connector_Generic:Conn_01x01
- added J8: Conn_01x06, Connector_PinHeader_1.00mm:PinHeader_1x06_P1.00mm_Vertical, symbol Connector_Generic:Conn_01x06
- added Q2: DTC143ZEBTL, DTC:SOTFL50P160X85-3N, symbol DTC:DTC143ZEBTL
- added R32: 100k, Resistor_SMD:R_0805_2012Metric, symbol Device:R_Small
- added R36: 1K, Resistor_SMD:R_0805_2012Metric, symbol Device:R_Small
- added R50, R51: 100R, Resistor_SMD:R_0805_2012Metric, symbol Device:R_Small
- added S1: SLW-12689-4A-N-D, SLW12689:SLW126894AND, symbol switch:SLW-12689-4A-N-D
- added U19: L86-M33, GPS:L80-M39, symbol GPS:L86-M33
- added U20: AO3407A, AO3407A:SOT-23-3L_AOS, symbol AO3407A:AO3407A
- R22: value 10K -> 100K
Connections:
- net +5V: now also R22.1, S1.3
- net GND: now also J3.1, J3.2, U10.52 (GND), C37.1, C42.2, C45.1, Q2.2 (E), S1.1, S1.4 (MH1), S1.5 (MH2), U19.12 (GND_2), U19.3 (GND_1); no longer R22.2
- net GPS_EN: now also J8.4 (Pin_4)
- net GPS_ON: now also J8.5 (Pin_5), R32.2, U20.1 (G)
- net GPS_PWR: now also J8.6 (Pin_6), R32.1, U20.2 (S)
- net RXGPS: now also J8.3 (Pin_3), R50.2
- net TMPPS: now also J8.1 (Pin_1), U19.6 (1PPS)
- net TXGPS: now also J8.2 (Pin_2), R51.2
- net at U11.4 (/CE): now also R22.2, S1.2; no longer R22.1
- net at U11.7 (ILIM/VSET): now also S2.2, C37.2
- net GPS_RTC renamed GPS_BCK_PW
- net GPS_BCK_PW: now also C42.1, C45.2, U19.5 (V_BCKP)
- net antenna renamed Antenna
- net Antenna: now also U19.11 (EX_ANT)
- new net: Q2.1 (B), U19.8 (AADET_N)
- new net: Q2.3 (C), R36.1
- new net: J13.1 (Pin_1), U19.7 (FORCE_ON)
- new net: CHG2.1 (K), R36.2
- new net: R51.1, U19.2 (TXD1)
- new net: R50.1, U19.1 (RXD1)
- new net GPS_PWR_M: CHG2.2 (A), U19.10 (RESET), U19.4 (VCC), U20.3 (D)
- no-connect marks 55 -> 45
Other:
- note added: "6.8KΩ = 4.05V / 1A (Sodium battery) 5.1KΩ = 3.65V / 1A (LiFePO4 battery)"
- note added: "Energy intake, solar, battery and battery charging module Solar and battery charging module"
- note added: "Microcontrollers"
- note added: "Mounting"
- note added: "Recharge battery (GN) or not (SYS)"
- note removed: "5.1KΩ = 3.65V / 1A 6.8KΩ = 4.05V / 1A"
- note removed: "GNSS (GPS)"
- note removed: "Micro controllers"
- note removed: "Solar and battery charging module"
- moved on the sheet: BAT1, C27, C28, C29, C32, C40, C41, CHG1, D1, D2, D5, F3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
